File: controller-pcb/stringlight-usb.kicad_pcb (KiCad board)
At the start: 2 copper layers, 87.7 x 49.7 mm, 45 parts, among them J1 USB_B, J2 Conn_01x05, J3 Screw_Terminal_01x03, J4 Screw_Terminal_01x03, Q2 BC817, Q3 MJD31, Q4 MJD31, Q5 BC817, U1 PSSI2021SAY, U2 MCP1703Ax-330xxTT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

Commit message: enclosure
Other:
- board text added: "enclosure: Euroclamp CEM17-S1-GY"
Changed lines of the file:
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@@
 		(layer "Edge.Cuts")
+	)
+	(gr_text "enclosure: Euroclamp CEM17-S1-GY"
+		(at 73.75 119 0)
+		(layer "Cmts.User")
+		(effects
+			(font
+				(size 1 1)
+				(thickness 0.15)
+			)
+			(justify left bottom)
+		)
 	)
 	(segment

Commit message: - speed up opto RX with additional 1k resistor - add firmware-based 24V-data short circuit protection (goes into fault mode)
Parts:
- added R14: 1k, Resistor_SMD:R_0603_1608Metric_Pad0.98x0.95mm_HandSolder, F.Cu at (96.4, 161.5)
- added R15: 1k, Resistor_SMD:R_0603_1608Metric_Pad0.98x0.95mm_HandSolder, F.Cu at (90.1, 149.0)
- J3, J4: value Screw_Terminal_01x03 -> ML253-5-D-LC-BK
Routing:
- net Net-(R15-Pad2): track 2.94 -> 5.97 mm
- net Net-(R14-Pad2): track 8.37 -> 10.3 mm
- net /2_GND: track 40.0 -> 41.7 mm
- net /1_GND: track 36.3 -> 37.7 mm
